File: spresense_payload.kicad_pcb (KiCad board)
At the start: 4 copper layers, 88 x 94.5 mm, 80 parts, among them J1 Conn_01x02_Pin, J2 Conn_01x02_Pin, J3 Life Makes Lemonade, J4 Conn_02x02_Odd_Even, J9 Conn_01x02_Pin, U1 W25Q128JVS, U10 DRV8212PDSGR, U11 TPS62913, U12 TPS62143RGTR, U13 TPS22993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

Commit message: changed mounting holes
Parts:
- removed C50: 220nf, Capacitor_SMD:C_0402_1005Metric
- removed C51, C53: 100nf, Capacitor_SMD:C_0402_1005Metric
- removed J3: Life Makes Lemonade, Connector_PinHeader_2.54mm:PinHeader_1x06_P2.54mm_Vertical
- removed J4: Conn_02x02_Odd_Even, Connector_Hirose:Hirose_DF11-4DP-2DSA_2x02_P2.00mm_Vertical
- removed U13: TPS22993, Package_DFN_QFN:Texas_S-PWQFN-N20
- added C27: 220nF, Capacitor_SMD:C_0402_1005Metric, F.Cu at (239.9, 69.3)
- added C28: 100nF, Capacitor_SMD:C_0402_1005Metric, F.Cu at (239.7, 65.3)
- added C29: 100nF, Capacitor_SMD:C_0402_1005Metric, F.Cu at (241.7, 67.5)
- added C30: 10uF, Capacitor_SMD:C_0402_1005Metric, F.Cu at (242.9, 67.5)
- added CR1: CMS04TE12L_Q_M, footprints:M-FLAT_TOS, F.Cu at (254.6, 91.8)
- added CR2: CMS04TE12L_Q_M, footprints:M-FLAT_TOS, F.Cu at (242.5, 74.1)
- added J18: Payload, Connector_Hirose:Hirose_DF11-12DP-2DSA_2x06_P2.00mm_Vertical, F.Cu at (268.4, 81.8)
- H7, H8, H9: value MountingHole -> (none); footprint MountingHole:MountingHole_2.2mm_M2 -> (none)
- U3: value LSM303AGRTR -> LIS2MDLTR; footprint footprints:LGA12R50P_200X200X100 -> footprints:PQFN50P200X200X70-12N
- moved H10 79.7 mm to (272.9, 57.7)
- moved H3 74.5 mm to (208.3, 123.0), turned to 180 degrees
- moved H6 66.1 mm to (219.2, 123.0), turned to 90 degrees
- moved H9 52.6 mm to (208.3, 64.0), turned to 90 degrees
- moved H8 50.1 mm to (219.2, 64.0), turned to 90 degrees
- moved H5 5.75 mm to (213.9, 46.8)
- moved H7 4.42 mm to (272.9, 46.8)
- moved J2 3.74 mm to (269.6, 65.0)
- moved H4 2.98 mm to (213.9, 57.7), turned to 90 degrees
- moved U3 1.84 mm to (239.7, 67.3)
Connections:
- net VBUS renamed PAYLOAD_BATT
- C21 pad 1: +5V -> Net-(U12-FSW)
- L1 pad 1: +3.3V -> Net-(U11-VO)
- L2 pad 2: +5V -> Net-(U12-FSW)
- R14 pad 1: +3.3V -> Net-(U11-VO)
- R20 pad 1: +3.3V -> Net-(U11-VO)
- R21 pad 2: +5V -> Net-(U12-FSW)
- U11 pad 3: +3.3V -> Net-(U11-VO)
- U12 pad 14: +5V -> Net-(U12-FSW)
- U12 pad 7: +5V -> Net-(U12-FSW)
- U3 pad 2: +3.3V -> unconnected-(U3-NC1-Pad2)
Routing:
- net +5V: track 75.5 -> 47.5 mm, vias 8 -> 6
- net Net-(U12-FSW): track 0.00 -> 26.5 mm, vias 0 -> 2
- net SCL_FB: track 24.3 -> 0.00 mm
- net +3.3VA: track 21.2 -> 0.00 mm, vias 1 -> 0
- net SDA_FB: track 18.1 -> 0.00 mm
- net TX_FB: track 8.65 -> 22.0 mm
- net Net-(U11-VO): track 0.00 -> 13.1 mm
- net +3.3V: track 85.8 -> 79.3 mm
- net RX_FB: track 19.0 -> 22.0 mm
- net I2C_SCL: track 10.1 -> 12.4 mm
- net VBAT: track 2.00 -> 0.00 mm
- net PAYLOAD_PWR: track 0.00 -> 2.00 mm
- net GND: track 81.0 -> 79.4 mm, vias 59 -> 402
- net D08: track 19.9 -> 21.1 mm
- net Net-(J2-Pin_2): track 17.7 -> 16.8 mm
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- added copper zone on F.Cu, net +5V
- added copper zone on F.Cu, net Net-(U11-VO)
- removed copper zone on F.Cu, net VBAT
